File: PCB_DISENO/BOARD_ESP32_S3/BOARD_ESP32_S3.kicad_sch (KiCad schematic)
At the start: 48 parts, among them J1 INPUT_EXT, J2 USB_B_Micro, J3 CON TEST, J4 INPUT_EXT, Q1 Q_NPN_BEC, Q2 Q_NPN_BEC, U1 ESP32-S3-WROOM-1, U2 CH340C, U3 3v3 1A, U5 ACS712

Commit message: Se agregan elementos de maestria
Parts:
- added R11, R12: 10K, Resistor_SMD:R_0805_2012Metric, symbol Device:R_US
Connections:
- net GND: now also R12.1
- net GPIO01: now also U5.7 (VIOUT); no longer BUS_I2C1.4, EXTERNAL_I2C1.4
- net GPIO02: now also R11.1, R12.2; no longer BUS_I2C1.3, EXTERNAL_I2C1.3
- net GPIO36: now also BUS_I2C1.3, EXTERNAL_I2C1.3
- net GPIO37: now also BUS_I2C1.4, EXTERNAL_I2C1.4
- new net VBAT: R11.2
Other:
- moved on the sheet: D1, D2
